File: SPI2WS2812.kicad_pcb (KiCad board)
At the start: 2 copper layers, 61 x 40.6 mm, 19 parts, among them J1 Conn_01x05, J2 Conn_01x03, T1 2N7002, T2 2N7002, T3 2N7002, T4 BSS84

Commit message: git-svn-id: file:///D/00%20-%20Dev%20&%20Calculs/RepoTortoiseSVN_PCB/SPI2WS2812/trunk@11 14acadc8-6264-6a46-bd6b-d9c895d7e7fb
Parts:
- removed D1, D2: 1N6263, Diode_THT:D_DO-35_SOD27_P7.62mm_Horizontal
- added D12: BAT54S, Package_TO_SOT_SMD:SOT-23, F.Cu at (101.6, 81.3)
- C1, C2, C3, C4: footprint Capacitor_THT:C_Disc_D5.0mm_W2.5mm_P2.50mm -> Capacitor_SMD:C_1210_3225Metric_Pad1.33x2.70mm_HandSolder
- R1, R2, R4: footprint Resistor_THT:R_Axial_DIN0207_L6.3mm_D2.5mm_P10.16mm_Horizontal -> Resistor_SMD:R_1210_3225Metric_Pad1.30x2.65mm_HandSolder
- T1, T2, T3, T4: footprint Package_TO_SOT_THT:TO-92_Inline_Wide -> Package_TO_SOT_SMD:SOT-23_Handsoldering
- moved C4 23.3 mm to (129.5, 82.5)
- moved R1 20.4 mm to (96.5, 82.5), turned to 0 degrees
- moved T2 15.2 mm to (106.7, 88.9)
- moved T1 7.41 mm to (95.2, 77.5), turned to 0 degrees
- moved R4 6.36 mm to (91.2, 72.4), turned to 0 degrees
- moved T4 5.68 mm to (124.5, 73.7)
- moved C1 5.36 mm to (92.7, 87.6)
- moved R2 5.24 mm to (108.0, 71.1)
- moved J2 5.08 mm to (134.6, 81.3), turned to 180 degrees
- moved C3 3.81 mm to (100.3, 71.1)
- moved T3 2.54 mm to (124.5, 78.7)
Connections:
- C1 pad 2: Net-(C1-Pad2) -> Net-(T1-Pad3)
- R1 pad 1: Net-(D2-Pad2) -> /MOSI
- R1 pad 2: Net-(C1-Pad2) -> Net-(R1-Pad2)
- T1 pad 3: Net-(C1-Pad2) -> Net-(T1-Pad3)
- T2 pad 1: Net-(C1-Pad2) -> Net-(T1-Pad3)
Routing:
- net GND: track 0.00 -> 50.8 mm
- net Net-(C1-Pad2): track 43.2 -> 0.00 mm
- net Net-(T1-Pad3): track 0.00 -> 27.6 mm
- net Net-(D2-Pad2): track 19.0 -> 0.00 mm
- net /~{EN}: track 22.9 -> 14.9 mm
- net Net-(C2-Pad2): track 35.6 -> 43.1 mm
- net +5V: track 88.9 -> 82.3 mm
- net /DOUT: track 17.8 -> 13.7 mm
- net /SCK: track 7.64 -> 11.4 mm
- net Net-(R1-Pad2): track 0.00 -> 2.73 mm
- net /MOSI: track 11.4 -> 12.7 mm
- added copper zone on F.Cu, net GND

Commit message: git-svn-id: file:///D/00%20-%20Dev%20&%20Calculs/RepoTortoiseSVN_PCB/SPI2WS2812/trunk@12 14acadc8-6264-6a46-bd6b-d9c895d7e7fb
Parts:
- removed J1: Conn_01x05, Connector_PinHeader_2.54mm:PinHeader_1x05_P2.54mm_Vertical
- removed J2: Conn_01x03, Connector_PinHeader_2.54mm:PinHeader_1x03_P2.54mm_Vertical
- added J3: Conn_01x06, Connector_PinHeader_2.54mm:PinHeader_1x06_P2.54mm_Vertical, F.Cu at (119.4, 91.4)
- moved H1 48.5 mm to (88.9, 111.8), turned to 90 degrees
- moved H2 45.8 mm to (88.9, 61.0), turned to 90 degrees
- moved C2 41.3 mm to (95.9, 106.7)
- moved H3 39.8 mm to (119.4, 111.8), turned to 90 degrees
- moved H4 36.4 mm to (119.4, 61.0), turned to 90 degrees
- moved T3 35.7 mm to (96.5, 101.0)
- moved T4 35.3 mm to (96.5, 95.2)
- moved T1 34.1 mm to (111.8, 107.3), turned to 180 degrees
- moved C4 27.0 mm to (103.5, 89.5), turned to -90 degrees
- moved R4 25.4 mm to (109.9, 89.5), turned to 90 degrees
- moved C1 25.2 mm to (113.7, 101.6), turned to 180 degrees
- moved R2 24.3 mm to (92.1, 89.5), turned to -90 degrees
- moved R1 22.1 mm to (113.7, 96.5), turned to 180 degrees
- moved C3 18.6 mm to (97.8, 89.5), turned to -90 degrees
- moved D12 17.1 mm to (106.0, 97.8), turned to 180 degrees
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Routing:
- net GND: track 50.8 -> 0.00 mm
- net +5V: track 82.3 -> 38.0 mm
- net /~{EN}: track 14.9 -> 43.5 mm
- net Net-(C2-Pad2): track 43.1 -> 25.0 mm
- net /DOUT: track 13.7 -> 29.5 mm
- net /MOSI: track 12.7 -> 4.16 mm
- net /SCK: track 11.4 -> 5.20 mm
- net Net-(C1-Pad2): track 27.6 -> 21.7 mm
- net Net-(D12-Pad2): track 2.73 -> 5.27 mm
Other:
- board size 61 x 40.6 mm -> 40.6 x 61 mm

Commit message: git-svn-id: file:///D/00%20-%20Dev%20&%20Calculs/RepoTortoiseSVN_PCB/SPI2WS2812/trunk@13 14acadc8-6264-6a46-bd6b-d9c895d7e7fb
Parts:
- removed D12: BAT54S, Package_TO_SOT_SMD:SOT-23
- added C10: 1nF, Capacitor_SMD:C_1210_3225Metric_Pad1.33x2.70mm_HandSolder, B.Cu at (111.8, 106.7)
- added C11: 10nF, Capacitor_SMD:C_1210_3225Metric_Pad1.33x2.70mm_HandSolder, B.Cu at (104.1, 90.2)
- added C12: 1µF, Capacitor_SMD:C_1210_3225Metric_Pad1.33x2.70mm_HandSolder, B.Cu at (98.4, 90.2)
- added C13: 1nF, Capacitor_SMD:C_1210_3225Metric_Pad1.33x2.70mm_HandSolder, B.Cu at (114.3, 71.1)
- added C14: 1nF, Capacitor_SMD:C_1210_3225Metric_Pad1.33x2.70mm_HandSolder, B.Cu at (97.2, 66.0)
- added C15: 10nF, Capacitor_SMD:C_1210_3225Metric_Pad1.33x2.70mm_HandSolder, B.Cu at (104.1, 82.5)
- added C16: 1µF, Capacitor_SMD:C_1210_3225Metric_Pad1.33x2.70mm_HandSolder, B.Cu at (109.2, 82.5)
- added C5: 1nF, Capacitor_SMD:C_1210_3225Metric_Pad1.33x2.70mm_HandSolder, F.Cu at (94.6, 71.1)
- added C6: 1nF, Capacitor_SMD:C_1210_3225Metric_Pad1.33x2.70mm_HandSolder, F.Cu at (112.4, 66.0)
- added C7: 10nF, Capacitor_SMD:C_1210_3225Metric_Pad1.33x2.70mm_HandSolder, F.Cu at (104.1, 82.5)
- added C8: 1µF, Capacitor_SMD:C_1210_3225Metric_Pad1.33x2.70mm_HandSolder, F.Cu at (99.1, 82.5)
- added C9: 1nF, Capacitor_SMD:C_1210_3225Metric_Pad1.33x2.70mm_HandSolder, B.Cu at (94.0, 101.6)
- added D1: BAT54S, Package_TO_SOT_SMD:SOT-23, F.Cu at (106.0, 97.8)
- added D2: BAT54S, Package_TO_SOT_SMD:SOT-23, F.Cu at (102.2, 74.9)
- added D3: BAT54S, Package_TO_SOT_SMD:SOT-23, B.Cu at (101.9, 97.8)
- added D4: BAT54S, Package_TO_SOT_SMD:SOT-23, B.Cu at (105.1, 74.9)
- added J1: Conn_01x06, Connector_PinHeader_2.54mm:PinHeader_1x06_P2.54mm_Vertical, F.Cu at (88.9, 81.3)
- added J2: Conn_01x06, Connector_PinHeader_2.54mm:PinHeader_1x06_P2.54mm_Vertical, B.Cu at (88.9, 91.4)
- added J4: Conn_01x06, Connector_PinHeader_2.54mm:PinHeader_1x06_P2.54mm_Vertical, B.Cu at (119.4, 81.3)
- added R10: 220 Ohm, Resistor_SMD:R_1210_3225Metric_Pad1.30x2.65mm_HandSolder, B.Cu at (114.3, 76.2)
- added R11: 1M, Resistor_SMD:R_1210_3225Metric_Pad1.30x2.65mm_HandSolder, B.Cu at (114.9, 82.5)
- added R12: 220 Ohm, Resistor_SMD:R_1210_3225Metric_Pad1.30x2.65mm_HandSolder, B.Cu at (97.2, 82.5)
- added R3: 220 Ohm, Resistor_SMD:R_1210_3225Metric_Pad1.30x2.65mm_HandSolder, F.Cu at (96.5, 90.2)
- added R5: 1M, Resistor_SMD:R_1210_3225Metric_Pad1.30x2.65mm_HandSolder, F.Cu at (94.0, 82.5)
- added R6: 220 Ohm, Resistor_SMD:R_1210_3225Metric_Pad1.30x2.65mm_HandSolder, F.Cu at (111.8, 82.5)
- added R7: 220 Ohm, Resistor_SMD:R_1210_3225Metric_Pad1.30x2.65mm_HandSolder, B.Cu at (94.0, 96.5)
- added R8: 1M, Resistor_SMD:R_1210_3225Metric_Pad1.30x2.65mm_HandSolder, B.Cu at (93.3, 90.2)
- added R9: 220 Ohm, Resistor_SMD:R_1210_3225Metric_Pad1.30x2.65mm_HandSolder, B.Cu at (111.8, 90.2)
- added T10: 2N7002, Package_TO_SOT_SMD:SOT-23_Handsoldering, B.Cu at (104.8, 104.8)
- added T11: BSS84, Package_TO_SOT_SMD:SOT-23_Handsoldering, B.Cu at (111.8, 94.6)
- added T12: 2N7002, Package_TO_SOT_SMD:SOT-23_Handsoldering, B.Cu at (111.8, 100.3)
- added T13: 2N7002, Package_TO_SOT_SMD:SOT-23_Handsoldering, B.Cu at (112.4, 65.4)
- added T14: 2N7002, Package_TO_SOT_SMD:SOT-23_Handsoldering, B.Cu at (104.1, 67.9)
- added T15: BSS84, Package_TO_SOT_SMD:SOT-23_Handsoldering, B.Cu at (97.2, 78.1)
- added T16: 2N7002, Package_TO_SOT_SMD:SOT-23_Handsoldering, B.Cu at (97.2, 72.4)
- added T5: 2N7002, Package_TO_SOT_SMD:SOT-23_Handsoldering, F.Cu at (96.5, 65.4)
- added T6: 2N7002, Package_TO_SOT_SMD:SOT-23_Handsoldering, F.Cu at (105.4, 67.9)
- added T7: BSS84, Package_TO_SOT_SMD:SOT-23_Handsoldering, F.Cu at (111.8, 78.1)
- added T8: 2N7002, Package_TO_SOT_SMD:SOT-23_Handsoldering, F.Cu at (111.8, 72.4)
- added T9: 2N7002, Package_TO_SOT_SMD:SOT-23_Handsoldering, B.Cu at (95.2, 107.3)
- R2: value 220 Ohm -> 1M
- R4: value 1M -> 220 Ohm
- T3: value 2N7002 -> BSS84
- T4: value BSS84 -> 2N7002
- moved R2 22.2 mm to (114.3, 90.2), turned to 90 degrees
- moved R4 20.3 mm to (94.6, 76.2), turned to 0 degrees
- moved C3 6.38 mm to (104.1, 90.2)
- moved C4 5.75 mm to (109.2, 90.2)
- moved T3 5.72 mm to (96.5, 95.2)
- moved T4 5.72 mm to (96.5, 101.0)
Connections:
- net /DOUT renamed /DOUT_0
- net /MOSI renamed /MOSI_0
- net /SCK renamed /SCK_0
- C2 pad 1: GND -> /GND0
- C3 pad 1: GND -> /GND0
- C3 pad 2: +5V -> /+5V0
- C4 pad 1: GND -> /GND0
- C4 pad 2: +5V -> /+5V0
- H1 pad 1: GND -> /GND2
- H2 pad 1: GND -> /GND1
- H3 pad 1: GND -> /GND0
- H4 pad 1: GND -> /GND3
- J3 pad 1: +5V -> /+5V0
- J3 pad 5: /~{EN} -> /~{EN}_0
- J3 pad 6: GND -> /GND0
- R2 pad 1: +5V -> /+5V0
- R2 pad 2: Net-(C2-Pad2) -> /~{EN}_0
- R4 pad 1: +5V -> /MOSI_1
- R4 pad 2: /~{EN} -> Net-(D2-Pad2)
- T1 pad 1: /~{EN} -> /~{EN}_0
- T1 pad 2: GND -> /GND0
- T2 pad 2: GND -> /GND0
- T3 pad 2: GND -> /+5V0
- T4 pad 2: +5V -> /GND0
Routing:
- net /~{EN}: track 43.5 -> 0.00 mm
- net /~{EN}_1: track 0.00 -> 38.9 mm
- net /~{EN}_0: track 0.00 -> 38.1 mm
- net +5V: track 38.0 -> 0.00 mm
- net /~{EN}_3: track 0.00 -> 35.9 mm
- net /~{EN}_2: track 0.00 -> 35.4 mm
- net /+5V0: track 0.00 -> 30.1 mm
- net /+5V1: track 0.00 -> 29.6 mm
- net /+5V2: track 0.00 -> 29.1 mm
- net /+5V3: track 0.00 -> 29.0 mm
- net /DOUT_2: track 0.00 -> 27.9 mm
- net /DOUT_1: track 0.00 -> 27.9 mm
- net /DOUT_3: track 0.00 -> 27.2 mm
- net Net-(C14-Pad2): track 0.00 -> 26.3 mm
- net Net-(C10-Pad2): track 0.00 -> 26.3 mm
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- added copper zone on B.Cu, net /GND0
- added copper zone on F.Cu, net /GND0
- added copper zone on B.Cu, net /GND1
- added copper zone on F.Cu, net /GND1
- added copper zone on B.Cu, net /GND2
- added copper zone on F.Cu, net /GND2
- added copper zone on B.Cu, net /GND3
- added copper zone on F.Cu, net /GND3
- removed copper zone on B.Cu, net GND
- removed copper zone on F.Cu, net GND
Other:
- board text added: "+"
- board text added: "1"
- board text added: "2"
- board text added: "3"
- board text added: "4"
- board text added: "DO"
- board text added: "SCK"
- board text added: "SI"
- board text added: "~{EN}"

Commit message: Bon pour fabrication. Il ne reste plus qu'à faire une release v1.0
git-svn-id: file:///D/00%20-%20Dev%20&%20Calculs/RepoTortoiseSVN_PCB/SPI2WS2812/trunk@16 14acadc8-6264-6a46-bd6b-d9c895d7e7fb
Parts:
- moved T9 1.27 mm to (96.5, 107.3)
- moved C14 1.27 mm to (95.9, 66.0)
- moved D4 0.97 mm to (106.0, 74.9)
- moved T15 0.90 mm to (96.5, 77.5)
- moved T16 0.90 mm to (96.5, 71.8)
- moved C9 0.64 mm to (94.6, 101.6)
- moved R7 0.64 mm to (94.6, 96.5)
- moved T12 0.64 mm to (111.8, 101.0)
- moved C12 0.64 mm to (99.1, 90.2)
- moved R10 0.64 mm to (113.7, 76.2)
- moved C10 0.64 mm to (112.4, 106.7)
- moved R12 0.64 mm to (96.5, 82.6)
- moved R11 0.64 mm to (114.3, 82.5)
- moved R8 0.64 mm to (94.0, 90.2)
- moved T7 0.64 mm to (111.8, 77.5)
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Routing:
- net Net-(C13-Pad2): track 25.0 -> 21.6 mm
- net /~{EN}_2: track 35.4 -> 38.4 mm
- net /~{EN}_3: track 35.9 -> 38.4 mm
- net Net-(D4-Pad2): track 6.87 -> 5.27 mm
- net /DOUT_3: track 27.2 -> 28.6 mm
- net /+5V3: track 29.0 -> 30.1 mm
- net /+5V2: track 29.1 -> 30.1 mm
- net /DOUT_1: track 27.9 -> 28.6 mm
- net /DOUT_2: track 27.9 -> 28.6 mm
- net Net-(C9-Pad2): track 22.4 -> 21.6 mm
- net Net-(C5-Pad2): track 22.3 -> 21.6 mm
- net /MOSI_2: track 3.53 -> 4.17 mm
- net /MOSI_3: track 3.53 -> 4.17 mm
- net /~{EN}_1: track 38.9 -> 38.4 mm
