File: SPI2WS2812.kicad_pcb (KiCad board)
At the start: 2 copper layers, 40.6 x 61 mm, 56 parts, among them J1 Conn_01x06, J2 Conn_01x06, J3 Conn_01x06, J4 Conn_01x06, T1 2N7002, T10 2N7002, T11 BSS84, T12 2N7002, T13 2N7002, T14 2N7002, T15 BSS84, T16 2N7002, T2 2N7002, T3 BSS84, T4 2N7002, T5 2N7002, T6 2N7002, T7 BSS84, T8 2N7002, T9 2N7002

Commit message: Avec les réglages "Rancunes"
git-svn-id: file:///D/00%20-%20Dev%20&%20Calculs/RepoTortoiseSVN_PCB/SPI2WS2812/trunk@19 14acadc8-6264-6a46-bd6b-d9c895d7e7fb
Other:
- rule pad_to_mask_clearance: 0 -> 0.1
Changed lines of the file:
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@@
       (dielectric_constraints no)
     )
-    (pad_to_mask_clearance 0)
+    (pad_to_mask_clearance 0.1)
+    (pad_to_paste_clearance_ratio -0.1)
     (pcbplotparams
       (layerselection 0x00010fc_ffffffff)
@@
     (pts (xy 88.9 116.84) (xy 88.9 55.88))
     (height -12.7)
-    (gr_text "60.9600 mm" (at 75.05 86.36 90) (layer "User.2")
+    (gr_text "60,9600 mm" (at 75.05 86.36 90) (layer "User.2")
       (effects (font (size 1 1) (thickness 0.15)))
     )
@@
     (pts (xy 83.82 60.96) (xy 124.46 60.96))
     (height -12.7)
-    (gr_text "40.6400 mm" (at 104.14 47.11) (layer "User.2")
+    (gr_text "40,6400 mm" (at 104.14 47.11) (layer "User.2")
       (effects (font (size 1 1) (thickness 0.15)))
     )
@@
     (pts (xy 83.82 86.36) (xy 83.82 116.84))
     (height 3.175)
-    (gr_text "30.4800 mm" (at 79.495 101.6 90) (layer "User.2")
+    (gr_text "30,4800 mm" (at 79.495 101.6 90) (layer "User.2")
       (effects (font (size 1 1) (thickness 0.15)))
     )
@@
     (pts (xy 83.82 86.36) (xy 83.82 55.88))
     (height -13.335)
-    (gr_text "30.4800 mm" (at 69.335 71.12 90) (layer "User.2")
-      (effects (font (size 1 1) (thickness 0.15)))
-    )
+    (gr_text "30,4800 mm" (at 69.335 71.12 90) (layer "User.2")
+      (effects (font (size 1 1) (thickness 0.15)))
+    )

Commit message: Allez on arrondi les angles
git-svn-id: file:///D/00%20-%20Dev%20&%20Calculs/RepoTortoiseSVN_PCB/SPI2WS2812/trunk@20 14acadc8-6264-6a46-bd6b-d9c895d7e7fb
Routing:
- net Net-(C13-Pad2): track 21.6 -> 24.1 mm
- net Net-(C9-Pad2): track 21.6 -> 24.1 mm
- net Net-(C5-Pad2): track 21.6 -> 23.8 mm
- net Net-(C1-Pad2): track 21.6 -> 23.8 mm
- net /~{EN}_1: track 38.4 -> 38.9 mm
- net /~{EN}_2: track 38.4 -> 38.9 mm
- net /~{EN}_3: track 38.4 -> 38.9 mm

Commit message: git-svn-id: file:///D/00%20-%20Dev%20&%20Calculs/RepoTortoiseSVN_PCB/SPI2WS2812/trunk@23 14acadc8-6264-6a46-bd6b-d9c895d7e7fb
Parts:
- D1, D2, D3, D4: value BAT54S -> BAS40-04
Changed lines of the file:
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@@
   (net 2 "/GND0")
   (net 3 "Net-(C1-Pad2)")
-  (net 4 "Net-(D1-Pad2)")
+  (net 4 "Net-(R1-Pad2)")
   (net 5 "/SCK_0")
   (net 6 "/SCK_1")
@@
   (net 13 "Net-(C13-Pad2)")
   (net 14 "Net-(C14-Pad2)")
-  (net 15 "Net-(D2-Pad2)")
-  (net 16 "Net-(D3-Pad2)")
-  (net 17 "Net-(D4-Pad2)")
+  (net 15 "Net-(R4-Pad2)")
+  (net 16 "Net-(R7-Pad2)")
+  (net 17 "Net-(R10-Pad2)")
   (net 18 "/DOUT_1")
   (net 19 "/MOSI_1")
@@
       (effects (font (size 1 1) (thickness 0.15)))
     )
-    (fp_text value "BAT54S" (at 0 2.4) (layer "F.Fab")
+    (fp_text value "BAS40-04" (at 0 2.4) (layer "F.Fab")
       (effects (font (size 1 1) (thickness 0.15)))
     )
@@
       (net 2 "/GND0") (pintype "passive"))
     (pad "2" smd roundrect (at -0.9375 0.95 180) (size 1.475 0.6) (layers "F.Cu" "F.Paste" "F.Mask") (roundrect_rratio 0.25)
-      (net 4 "Net-(D1-Pad2)") (pintype "passive"))
+      (net 4 "Net-(R1-Pad2)") (pintype "passive"))
     (pad "3" smd roundrect (at 0.9375 0 180) (size 1.475 0.6) (layers "F.Cu" "F.Paste" "F.Mask") (roundrect_rratio 0.25)
       (net 3 "Net-(C1-Pad2)") (pintype "passive"))
@@
       (net 19 "/MOSI_1") (pintype "passive"))
     (pad "2" smd roundrect (at 1.55 0) (size 1.3 2.65) (layers "F.Cu" "F.Paste" "F.Mask") (roundrect_rratio 0.1923076923)
-      (net 15 "Net-(D2-Pad2)") (pintype "passive"))
+      (net 15 "Net-(R4-Pad2)") (pintype "passive"))
     (model "${KICAD6_3DMODEL_DIR}/Resistor_SMD.3dshapes/R_1210_3225Metric.wrl"
       (offset (xyz 0 0 0))
@@
       (effects (font (size 1 1) (thickness 0.15)))
     )
-    (fp_text value "BAT54S" (at 0 2.4 -180) (layer "F.Fab")
-      (effects (font (size 1 1) (thickness 0.15)))
-    )
-    (fp_text user "${REFERENCE}" (at 0 0 -180) (layer "F.Fab")
+    (fp_text value "BAS40-04" (at 0 2.4 -180) (layer "F.Fab")
+      (effects (font (size 1 1) (thickness 0.15)))
+    )
+    (fp_text user "${REFERENCE}" (at -0.635 0 -180) (layer "F.Fab")
       (effects (font (size 0.32 0.32) (thickness 0.05)))
     )
@@
       (net 31 "/GND1") (pintype "passive"))
     (pad "2" smd roundrect (at -0.9375 0.95) (size 1.475 0.6) (layers "F.Cu" "F.Paste" "F.Mask") (roundrect_rratio 0.25)
-      (net 15 "Net-(D2-Pad2)") (pintype "passive"))
+      (net 15 "Net-(R4-Pad2)") (pintype "passive"))
     (pad "3" smd roundrect (at 0.9375 0) (size 1.475 0.6) (layers "F.Cu" "F.Paste" "F.Mask") (roundrect_rratio 0.25)
       (net 7 "Net-(C5-Pad2)") (pintype "passive"))
@@
       (net 25 "/MOSI_0") (pintype "passive"))
     (pad "2" smd roundrect (at 1.55 0 180) (size 1.3 2.65) (layers "F.Cu" "F.Paste" "F.Mask") (roundrect_rratio 0.1923076923)
-      (net 4 "Net-(D1-Pad2)") (pintype "passive"))
+      (net 4 "Net-(R1-Pad2)") (pintype "passive"))
     (model "${KICAD6_3DMODEL_DIR}/Resistor_SMD.3dshapes/R_1210_3225Metric.wrl"
       (offset (xyz 0 0 0))
@@
       (effects (font (size 1 1) (thickness 0.15)) (justify mirror))
     )
-    (fp_text value "BAT54S" (at 0 -2.4) (layer "B.Fab")
+    (fp_text value "BAS40-04" (at 0 -2.4) (layer "B.Fab")
       (effects (font (size 1 1) (thickness 0.15)) (justify mirror))
     )
@@
       (net 33 "/GND2") (pintype "passive"))
     (pad "2" smd roundrect (at -0.9375 -0.95) (size 1.475 0.6) (layers "B.Cu" "B.Paste" "B.Mask") (roundrect_rratio 0.25)
-      (net 16 "Net-(D3-Pad2)") (pintype "passive"))
+      (net 16 "Net-(R7-Pad2)") (pintype "passive"))
     (pad "3" smd roundrect (at 0.9375 0) (size 1.475 0.6) (layers "B.Cu" "B.Paste" "B.Mask") (roundrect_rratio 0.25)
       (net 10 "Net-(C9-Pad2)") (pintype "passive"))
@@
       (effects (font (size 1 1) (thickness 0.15)) (justify mirror))
     )
-    (fp_text value "BAT54S" (at 0 -2.4) (layer "B.Fab")
+    (fp_text value "BAS40-04" (at 0 -2.4) (layer "B.Fab")
       (effects (font (size 1 1) (thickness 0.15)) (justify mirror))
     )
@@
       (net 35 "/GND3") (pintype "passive"))
     (pad "2" smd roundrect (at -0.9375 -0.95 180) (size 1.475 0.6) (layers "B.Cu" "B.Paste" "B.Mask") (roundrect_rratio 0.25)
-      (net 17 "Net-(D4-Pad2)") (pintype "passive"))
+      (net 17 "Net-(R10-Pad2)") (pintype "passive"))
     (pad "3" smd roundrect (at 0.9375 0 180) (size 1.475 0.6) (layers "B.Cu" "B.Paste" "B.Mask") (roundrect_rratio 0.25)
       (net 13 "Net-(C13-Pad2)") (pintype "passive"))
@@
       (net 22 "/MOSI_2") (pintype "passive"))
     (pad "2" smd roundrect (at 1.55 0) (size 1.3 2.65) (layers "B.Cu" "B.Paste" "B.Mask") (roundrect_rratio 0.1923076923)
-      (net 16 "Net-(D3-Pad2)") (pintype "passive"))
+      (net 16 "Net-(R7-Pad2)") (pintype "passive"))
     (model "${KICAD6_3DMODEL_DIR}/Resistor_SMD.3dshapes/R_1210_3225Metric.wrl"
       (offset (xyz 0 0 0))
@@
       (net 28 "/MOSI_3") (pintype "passive"))
     (pad "2" smd roundrect (at 1.55 0 180) (size 1.3 2.65) (layers "B.Cu" "B.Paste" "B.Mask") (roundrect_rratio 0.1923076923)
-      (net 17 "Net-(D4-Pad2)") (pintype "passive"))
+      (net 17 "Net-(R10-Pad2)") (pintype "passive"))
     (model "${KICAD6_3DMODEL_DIR}/Resistor_SMD.3dshapes/R_1210_3225Metric.wrl"
       (offset (xyz 0 0 0))
