File: SPI2WS2812.kicad_sch (KiCad schematic)
At the start: 19 parts, among them J1 Conn_01x05, J2 Conn_01x03, T1 2N7002, T2 2N7002, T3 2N7002, T4 BSS84

Commit message: git-svn-id: file:///D/00%20-%20Dev%20&%20Calculs/RepoTortoiseSVN_PCB/SPI2WS2812/trunk@11 14acadc8-6264-6a46-bd6b-d9c895d7e7fb
Parts:
- removed D1, D2: 1N6263, Diode_THT:D_DO-35_SOD27_P7.62mm_Horizontal, symbol Diode:1N6263
- added D12: BAT54S, Package_TO_SOT_SMD:SOT-23, symbol Diode:BAT54S
- C1, C2, C3, C4: footprint Capacitor_THT:C_Disc_D5.0mm_W2.5mm_P2.50mm -> Capacitor_SMD:C_1210_3225Metric_Pad1.33x2.70mm_HandSolder
- R1, R2, R4: footprint Resistor_THT:R_Axial_DIN0207_L6.3mm_D2.5mm_P10.16mm_Horizontal -> Resistor_SMD:R_1210_3225Metric_Pad1.30x2.65mm_HandSolder
- T1, T2, T3, T4: footprint Package_TO_SOT_THT:TO-92_Inline_Wide -> Package_TO_SOT_SMD:SOT-23_Handsoldering
Connections:
- net GND: now also D12.1
- net MOSI: now also R1.1
- net at C1.2, T1.3 (D), T2.1 (G): now also D12.3; no longer R1.2
- new net: D12.2, R1.2
Other:
- moved on the sheet: R1

Commit message: git-svn-id: file:///D/00%20-%20Dev%20&%20Calculs/RepoTortoiseSVN_PCB/SPI2WS2812/trunk@12 14acadc8-6264-6a46-bd6b-d9c895d7e7fb
Parts:
- removed J1: Conn_01x05, Connector_PinHeader_2.54mm:PinHeader_1x05_P2.54mm_Vertical, symbol Connector_Generic:Conn_01x05
- removed J2: Conn_01x03, Connector_PinHeader_2.54mm:PinHeader_1x03_P2.54mm_Vertical, symbol Connector_Generic:Conn_01x03
- added J3: Conn_01x06, Connector_PinHeader_2.54mm:PinHeader_1x06_P2.54mm_Vertical, symbol Connector_Generic:Conn_01x06
Connections:
- net +5V: now also J3.1 (Pin_1)
- net DOUT: now also J3.2 (Pin_2)
- net GND: now also J3.6 (Pin_6)
- net MOSI: now also J3.3 (Pin_3)
- net SCK: now also J3.4 (Pin_4)
- net ~{EN}: now also J3.5 (Pin_5)
Other:
- moved on the sheet: C3, C4

Commit message: git-svn-id: file:///D/00%20-%20Dev%20&%20Calculs/RepoTortoiseSVN_PCB/SPI2WS2812/trunk@13 14acadc8-6264-6a46-bd6b-d9c895d7e7fb
Parts:
- removed C1, C2: 1nF, Capacitor_SMD:C_1210_3225Metric_Pad1.33x2.70mm_HandSolder, symbol Device:C_Small
- removed C3: 10nF, Capacitor_SMD:C_1210_3225Metric_Pad1.33x2.70mm_HandSolder, symbol Device:C_Small
- removed C4: 1µF, Capacitor_SMD:C_1210_3225Metric_Pad1.33x2.70mm_HandSolder, symbol Device:C_Small
- removed D12: BAT54S, Package_TO_SOT_SMD:SOT-23, symbol Diode:BAT54S
- removed R1, R2: 220 Ohm, Resistor_SMD:R_1210_3225Metric_Pad1.30x2.65mm_HandSolder, symbol Device:R_Small
- removed R4: 1M, Resistor_SMD:R_1210_3225Metric_Pad1.30x2.65mm_HandSolder, symbol Device:R_Small
- removed T1, T2, T3: 2N7002, Package_TO_SOT_SMD:SOT-23_Handsoldering, symbol Transistor_FET:2N7002
- removed T4: BSS84, Package_TO_SOT_SMD:SOT-23_Handsoldering, symbol Transistor_FET:BSS84
- added J1, J2, J4: Conn_01x06, Connector_PinHeader_2.54mm:PinHeader_1x06_P2.54mm_Vertical, symbol Connector_Generic:Conn_01x06
Connections:
- net +5V renamed +5V0
- net DOUT renamed DOUT_0
- removed net GND: H1.1, H2.1, H3.1, H4.1, J3.6 (Pin_6)
- net MOSI renamed MOSI_0
- net SCK renamed SCK_0
- net ~{EN} renamed ~{EN}_0
- new net +5V1: J1.1 (Pin_1)
- new net +5V2: J2.1 (Pin_1)
- new net +5V3: J4.1 (Pin_1)
- new net DOUT_1: J1.2 (Pin_2)
- new net DOUT_2: J2.2 (Pin_2)
- new net DOUT_3: J4.2 (Pin_2)
- new net GND0: H3.1, J3.6 (Pin_6)
- new net GND1: H2.1, J1.6 (Pin_6)
- new net GND2: H1.1, J2.6 (Pin_6)
- new net GND3: H4.1, J4.6 (Pin_6)
- new net MOSI_1: J1.3 (Pin_3)
- new net MOSI_2: J2.3 (Pin_3)
- new net MOSI_3: J4.3 (Pin_3)
- new net SCK_1: J1.4 (Pin_4)
- new net SCK_2: J2.4 (Pin_4)
- new net SCK_3: J4.4 (Pin_4)
- new net ~{EN}_1: J1.5 (Pin_5)
- new net ~{EN}_2: J2.5 (Pin_5)
- new net ~{EN}_3: J4.5 (Pin_5)
Other:
- added sheet Strip_WS2812_0 (Strip_WS2812.kicad_sch)
- added sheet Strip_WS2812_1 (Strip_WS2812.kicad_sch)
- added sheet Strip_WS2812_2 (Strip_WS2812.kicad_sch)
- added sheet Strip_WS2812_3 (Strip_WS2812.kicad_sch)
- moved on the sheet: J3
